File: Schematics/TeensyLev V2.sch (KiCad schematic (older format))
At the start: 14 parts, among them J1 Connector to transducers arra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, J1 Jack-DC, SW1 Power switch, U1 Teensy3.2, U2 Pololu TB6612FNG, U3 Adafruit 3321 miniTFTwithJoy, U4 Pololu S18V20ALV, U5 Pololu D24V10F5

Commit message: update
Other:
- note added: "See hack-S18V20ALV.png\nfor details"
Changed lines of the file:
@@
 EESchema Schematic File Version 4
-LIBS:TeensyLev V2-cache
 EELAYER 30 0
 EELAYER END
@@
 Wire Wire Line
 	2600 1400 2600 1550
+Text Notes 3100 3450 0    50   ~ 0
+See hack-S18V20ALV.png\nfor details
 $EndSCHEMATC
